Commit message: Lab 9: Vision-Based Target Tracking - Complete implementation with report

File: Week8/StudentTask.urdf (robot description, URDF)
Before this commit: robot my_custom_robot, 6 links, 5 joints
Links:
- added link caster_housing; visual cylinder length=0.028 radius=0.025; visual cylinder length=0.06 radius=0.01
- link caster_wheel: geometry visual sphere radius=0.02
Joints:
- added joint caster_housing_joint: type fixed, parent base_link, child caster_housing, origin xyz=0.15 0 0.1 rpy=0 0 0
- joint caster_wheel_joint: axis (none) -> 0 0 1; origin xyz=0.15 0 0.065 rpy=0 0 0 -> xyz=0 0 -0.08 rpy=0 0 0; parent base_link -> caster_housing; type fixed -> continuous
- joint left_wheel_joint: origin xyz=-0.1 0.17 0.07 rpy=1.5708 0 0 -> xyz=-0.1 0.19 0.07 rpy=1.5708 0 0
- joint right_wheel_joint: origin xyz=-0.1 -0.17 0.07 rpy=1.5708 0 0 -> xyz=-0.1 -0.19 0.07 rpy=1.5708 0 0
